File: Schematics/RejsaCAN v3.x (ESP32-S3 based board)/KiCad/RejsaCAN v3.4 - Schematic.kicad_pcb (KiCad board)
At the start: 4 copper layers, 63 x 49.5 mm, 87 parts, among them J1 Micro-Fit 3.0 4P R/A, J2 U.FL, J3 JST-XH 4P LTE, Q1 SS8050, U1 ESP32-S3-WROOM-1(N16R8), U2 SN65HVD230DR, U3 ME2807A33M3G, U4 LMR14006XDDCR, U5 MT9700, U6 CPC1018N, U7 LG290P03AAMD, U8 AP2112K-3.3

Commit message: PCB: move SPI1 (MTDO/MTCK/MTDI) out from under the WROOM into the header area
The recovered v3.4 placement had put the 3-pin SPI/JTAG header on three of
upstream's rear-access pads under the module (upstream's README: those pads
carry GPIO6/7/15/16, MTMS, PROG, JTAG_ENABLE, TXD0, RXD0 and have no
symbols, so they never entered this netlist; MISO/CLK/MOSI belong in the
header row). A header nobody can populate is a defect, so SPI1 now sits as a
second column beside GPIO1 (X 142.5, pins at 195.37/197.91/200.45), ~8 mm
from U1's MTDx pads, re-routed on B.Cu; the old under-module stubs are gone.
DRC: 0 errors, 0 unconnected.

Co-Authored-By: Claude Fable 5 <noreply@anthropic.com>
Parts:
- moved SPI1 23.2 mm to (142.5, 195.4)
Routing:
- net MTCK: track 38.0 -> 51.2 mm, vias 0 -> 2
- net MTDI: track 40.7 -> 53.3 mm, vias 2 -> 3
- net MTDO: track 35.4 -> 44.4 mm
- net GND: vias 101 -> 99

Commit message: PCB: sync 7 stale footprint Value fields from the schematic (U4/U6/L1/R9/R10/R20/D5)
Co-Authored-By: Claude Fable 5 <noreply@anthropic.com>
Parts:
- D5: value SS34 -> SS34 (DNP)
- L1: value 10uH -> 15uH
- R10: value 10K -> 22.1k
- R20: value 500 -> 390
- R9: value 33K -> 69.8k
- U4: value LMR14006XDDCR -> LMR51610XDBVR
- U6: value CPC1018N -> GAQY212GS
Changed lines of the file:
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@@
 			)
 		)
-		(property "Value" "CPC1018N"
+		(property "Value" "GAQY212GS"
 			(at 0 3 0)
 			(layer "F.Fab")
@@
 			)
 		)
-		(property "Value" "500"
+		(property "Value" "390"
 			(at 0 1.17 0)
 			(layer "F.Fab")
@@
 			)
 		)
-		(property "Value" "33K"
+		(property "Value" "69.8k"
 			(at 0 1.17 0)
 			(layer "F.Fab")
@@
 			)
 		)
-		(property "Value" "SS34"
+		(property "Value" "SS34 (DNP)"
 			(at 0 2.6 0)
 			(layer "F.Fab")
@@
 			)
 		)
-		(property "Value" "10K"
+		(property "Value" "22.1k"
 			(at 0 1.17 180)
 			(layer "F.Fab")
@@
 			)
 		)
-		(property "Value" "LMR14006XDDCR"
+		(property "Value" "LMR51610XDBVR"
 			(at 0 2.4 0)
 			(layer "F.Fab")
@@
 			)
 		)
-		(property "Value" "10uH"
+		(property "Value" "15uH"
 			(at 0 2.4 0)
 			(layer "F.Fab")

Commit message: BOM: verified, stocked LCSC part on every line; equivalents for the unstocked ones
Every symbol now carries Manufacturer Part / Manufacturer / Supplier Part
(LCSC C-number) checked against LCSC stock on 2026-08-18. Land patterns of
the substitutes were compared numerically (EasyEDA footprint API) where the
package mattered:

- SD-CARD1: ATOM MR01A-01211 (C479742, out of stock) -> SOFNG TF-015
  (C113206): identical TF-015-family land within 0.1 mm incl. the two 1.0 mm
  pegs; XYECONN/SHOU HAN clones put the pegs 0.35 mm further out.
- L1: no 15 uH with adequate Isat in the SLP6028S land at LCSC -> the
  upstream SLP6028S100MTT 10 uH (C254862, 2.2 A, 35 mR, exact land).
- L2: 68 nH LQW15AN out of stock -> LQW15AN47NJ00D 47 nH wirewound
  (C192855, 228k); the ferrite-core 68 nH parts (SRF 750-800 MHz) are
  useless at L1/L5.
- U8: AP2112K-3.3 has 5 pcs -> RT9013-33GB (C47773, same SOT-23-5 pinout,
  low noise/high PSRR).
- D6/D7: SS110 in SOD-123F only exists as SMAF at LCSC -> onsemi
  MBR1H100SFT3G SOD-123FL 100 V 1 A (C235757).
- D13: 0.5 pF ESD9L5.0ST5G (C82326); its SOD-923 pads sit inside the 0402 land.
- F1 0466002.NRHF 2 A/63 V fast (C3105); F3 Walter 1206T4A63V 4 A time-lag
  (C354899). C6 CL32B225KCJSNNE (C55151), C13 CL10B104KC8NNNC (C15725),
  D4 MDD SMAJ33CA (C115251), U4 C20539658, U6 AQY212GS C719745, J1 C122413,
  J2 U.FL-R-SMT-1(10) C88373 (the field used to hold a pin-header C-number),
  J3 B4B-XH-A C144395.
- U7 LG290P03AAMD: not at LCSC (DigiKey ~$71-81), field says so.

The stale copied fields (D13 = a Samsung capacitor, F1/F3 = the old 1812
PTC, U4 = LMR14006, C6/C13 wrong dielectrics) would have matched wrong parts
in a JLC BOM upload. PCB Value fields re-synced; DRC unchanged (0 errors).

Co-Authored-By: Claude Fable 5 <noreply@anthropic.com>
Parts:
- D13: value TVS_Cj0.6pF -> ESD9L5.0ST5G 0.5pF
- D6, D7: value SS110 -> MBR1H100SFT3G
- F1: value 1206TD-2A -> 2A 63V fast 1206
- F3: value 1206TD-4A -> 4A 63V time-lag 1206
- L1: value 15uH -> 10uH
- L2: value 68nH -> 47nH
- SD-CARD1: value MR01A-01211 -> TF-015
- U6: value GAQY212GS -> AQY212GS
- U8: value AP2112K-3.3 -> RT9013-33GB
Changed lines of the file:
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@@
 			)
 		)
-		(property "Value" "GAQY212GS"
+		(property "Value" "AQY212GS"
 			(at 0 3 0)
 			(layer "F.Fab")
@@
 			)
 		)
-		(property "Value" "1206TD-2A"
+		(property "Value" "2A 63V fast 1206"
 			(at 0 1.83 0)
 			(layer "F.Fab")
@@
 			)
 		)
-		(property "Value" "68nH"
+		(property "Value" "47nH"
 			(at 0 1.17 90)
 			(layer "F.Fab")
@@
 			)
 		)
-		(property "Value" "TVS_Cj0.6pF"
+		(property "Value" "ESD9L5.0ST5G 0.5pF"
 			(at 0 1.17 90)
 			(layer "F.Fab")
@@
 			)
 		)
-		(property "Value" "SS110"
+		(property "Value" "MBR1H100SFT3G"
 			(at 0 2.1 0)
 			(layer "F.Fab")
@@
 			)
 		)
-		(property "Value" "AP2112K-3.3"
+		(property "Value" "RT9013-33GB"
 			(at 0 2.4 0)
 			(layer "F.Fab")
@@
 			)
 		)
-		(property "Value" "SS110"
+		(property "Value" "MBR1H100SFT3G"
 			(at 0 2.1 180)
 			(layer "F.Fab")
@@
 			)
 		)
-		(property "Value" "1206TD-4A"
+		(property "Value" "4A 63V time-lag 1206"
 			(at 0 1.83 0)
 			(layer "F.Fab")
@@
 			)
 		)
-		(property "Value" "15uH"
+		(property "Value" "10uH"
 			(at 0 2.4 0)
 			(layer "F.Fab")
@@
 			)
 		)
-		(property "Value" "MR01A-01211"
+		(property "Value" "TF-015"
 			(at 0 -7.376 0)
 			(layer "B.Fab")
